File: secu3v.sch (KiCad schematic (older format))
At the start: 188 parts, among them IC1 ATMEGA1284-A, P1 HCCPHPE24BKA90, P2 CONN_01X16, P3 CONN_02X03, Q1 BC817, Q10 BC817, Q11 BC817, Q12 BC817, Q13 BC817, Q14 BC817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

Commit message: промежуточная точка - исправлено размещение отверстий и платы в корпусе
Connections:
- net +VS: now also P1.1B, P1.1C; no longer P1.8A, P1.8B
- net CE_OUT: now also P1.7C; no longer P1.5C
- net FAN_OUT: now also P1.7B; no longer P1.6B
- net FE_OUT: now also P1.6A; no longer P1.3A
- net GAS: now also P1.6C; no longer P1.4C
- net IE_OUT: now also P1.6B; no longer P1.2A
- net IGN_OUT1: now also P1.8A, P2.4 (P4); no longer P1.1B, P2.1 (P1)
- net IGN_OUT2: now also P1.8B, P2.3 (P3); no longer P1.1C, P2.2 (P2)
- net IGN_OUT3: now also P2.2 (P2); no longer P2.3 (P3)
- net IGN_OUT4: now also P2.1 (P1); no longer P2.4 (P4)
- net RX_IN: now also P1.2A; no longer P1.7B
- net STB_OUT: now also P1.7A; no longer P1.6A
- net TX_OUT: now also P1.3A; no longer P1.7A
- net sync1+: now also P1.4C; no longer P1.6C
- net sync1-: now also P1.5C; no longer P1.7C
